File: Hardware/esp32-thing.sch (EAGLE design)
At the start: 71 parts, among them Q1 2.5A/30V, Q2 MBT3904DW1T1, U1 MCP73831, U3 AP2112K-3.3V, U4 FT231XS, U5 W25Q32FVSS, Y1 26MHz, Y2 32.768kHz

Commit message: Fixing ESP32 pin map, re-routing RX, TX
Parts:
- removed U$1: ESP32, esp32-thing-temp:ESP32
- added C27: 3.3nF, SparkFun-Capacitors:3.3NF-0603-100V-10%
- added U$2: ESP32-2, esp32-thing-temp:ESP32-2
Connections:
- removed net 20: J2.16, U$1.(VSPID/HS2_DATA3)GPIO20
- removed net RES_14K: R2.2, U$1.RES_14K
- new net N$4: C27.2, R2.1, U$2.RES_14K
- net 0: now also U$2.(ADC2:1/TOUCH1/RTC11/CLK_OUT1)GPIO0; no longer U$1.(ADC2:1/TOUCH1/RTC11/CLK_OUT1)GPIO0
- net 12: now also U$2.(GPIO12/ADC2:5/TOUCH5/RTC15/SPIQ)MTDI; no longer U$1.(GPIO12/ADC2:5/TOUCH5/RTC15/SPIQ)MTDI
- net 13: now also U$2.(GPIO13/ADC2:4/TOUCH4/RTC14/SPID/U0CTS)MTCK; no longer U$1.(GPIO13/ADC2:4/TOUCH4/RTC14/SPID/U0CTS)MTCK
- net 14: now also U$2.(GPIO14/ADC2:6/TOUCH6/RTC16/SPICLK)MTMS; no longer U$1.(GPIO14/ADC2:6/TOUCH6/RTC16/SPICLK)MTMS
- net 15: now also U$2.(GPIO15/ADC2:3/TOUCH3/RTC13/SPICSO/U0RTS)MTDO; no longer U$1.(GPIO15/ADC2:3/TOUCH3/RTC13/SPICSO/U0RTS)MTDO
- net 16: now also U$2.(HS1_DATA4)GPIO16; no longer U$1.(HS1_DATA4)GPIO16
- net 17: now also U$2.(HS1_DATA5)GPIO17; no longer U$1.(HS1_DATA5)GPIO17
- net 18: now also U$2.(VSPICLK/HS1_DATA7)GPIO18; no longer U$1.(VSPICLK/HS1_DATA7)GPIO18
- net 19: now also U$2.(VSPIQ/HS2_DATA2)GPIO19; no longer U$1.(VSPIQ/HS2_DATA2)GPIO19
- net 2: now also U$2.(ADC2:2/TOUCH2/RTC12/SPIWP)GPIO2; no longer U$1.(ADC2:2/TOUCH2/RTC12/SPIWP)GPIO2
- net 21: now also J2.19, U$2.(VSPIHD/HS2_CMD)GPIO21; no longer J2.18, U$1.(VSPIHD/HS2_CMD)GPIO21
- net 22: now also J2.16, U$2.(VSPIWP/HS2_CLK)GPIO22; no longer J2.17, U$1.(VSPIWP/HS2_CLK)GPIO22
- net 23: now also U$2.GPIO23; no longer U$1.GPIO23
- net 25: now also U$2.(DAC1/ADC2:8/RTC6)GPIO25; no longer U$1.(DAC1/ADC2:8/RTC6)GPIO25
- net 26: now also U$2.(DAC2/ADC2:9/RTC7)GPIO26; no longer U$1.(DAC2/ADC2:9/RTC7)GPIO26
- net 27: now also U$2.(ADC2:7/TOUCH7/RTC17)GPIO27; no longer U$1.(ADC2:7/TOUCH7/RTC17)GPIO27
- net 3.3V: now also U$2.VDD3P3_CPU, U$2.VDD3P3_RTC, U$2.VDDA, U$2.VDDA3P3; no longer U$1.VDD3P3_CPU, U$1.VDD3P3_RTC, U$1.VDDA, U$1.VDDA3P3
- net 32K_XN: now also U$2.32K_XN(GPIO33/ADC1:5/TOUCH8/RTC8); no longer U$1.32K_XN(GPIO33/ADC1:5/TOUCH8/RTC8)
- net 32K_XP: now also U$2.32K_XP(GPIO32/ADC1:4/TOUCH9/RTC9); no longer U$1.32K_XP(GPIO32/ADC1:4/TOUCH9/RTC9)
- net 34: now also U$2.VDET_1(GPI34/ADC1:6); no longer U$1.VDET_1(GPI34/ADC1:6)
- net 35: now also U$2.VDET_2(GPI35/ADC1:7); no longer U$1.VDET_2(GPI35/ADC1:7)
- net 36: now also U$2.SENSOR_VP(GPI36/ADC1:0/RTC0); no longer U$1.SENSOR_VP(GPI36/ADC1:0/RTC0)
- net 37: now also U$2.SENSOR_CAPP(GPI37/ADC1:1/RTC1); no longer U$1.SENSOR_CAPP(GPI37/ADC1:1/RTC1)
- net 38: now also U$2.SENSOR_CAPN(GPI38/ADC1:2/RTC2); no longer U$1.SENSOR_CAPN(GPI38/ADC1:2/RTC2)
- net 39: now also U$2.SENSOR_VN(GPI39/ADC1:3/RTC3); no longer U$1.SENSOR_VN(GPI39/ADC1:3/RTC3)
- net 4: now also U$2.(ADC2:0/TOUCH0/RTC10/SPIHD)GPIO4; no longer U$1.(ADC2:0/TOUCH0/RTC10/SPIHD)GPIO4
- net 5: now also U$2.(VSPICS0/HS1_DATA6)GPIO5; no longer U$1.(VSPICS0/HS1_DATA6)GPIO5
- net CAP_10N: now also C27.1, R2.2, U$2.CAP_10N; no longer U$1.CAP_10N
- net CHIP_PU: now also U$2.CHIP_PU; no longer U$1.CHIP_PU
- net FLASH_SCK: now also U$2.(GPIO6/SPICLK/HS1_CLK/U1CTS)SD_CLK; no longer U$1.(GPIO6/SPICLK/HS1_CLK/U1CTS)SD_CLK
- net FLASH_SCS: now also U$2.(GPIO11/SPICSO/HS1_CMD/U1RTS)SD_CMD; no longer U$1.(GPIO11/SPICSO/HS1_CMD/U1RTS)SD_CMD
- net FLASH_SDI: now also U$2.(GPIO8/SPID/HS1_DATA1)SD_DATA1; no longer U$1.(GPIO8/SPID/HS1_DATA1)SD_DATA1
- net FLASH_SDO: now also U$2.(GPIO7/SPI1/HS1_DATA0)SD_DATA0; no longer U$1.(GPIO7/SPI1/HS1_DATA0)SD_DATA0
- net FLASH_SHD: now also U$2.(GPIO9/SPIHD/HS1_DATA2/U1RX)SD_DATA2; no longer U$1.(GPIO9/SPIHD/HS1_DATA2/U1RX)SD_DATA2
- net FLASH_SWP: now also U$2.(GPIO10/SPIWP/HS1_DATA3/U1TX)SD_DATA3; no longer U$1.(GPIO10/SPIWP/HS1_DATA3/U1TX)SD_DATA3
- net FLASH_VDD: now also U$2.VDD3P3_SDIO; no longer U$1.VDD3P3_SDIO
- net GND: now also J2.20, U$2.GND; no longer R2.1, U$1.GND
- net LNA_IN: now also U$2.LNA_IN; no longer U$1.LNA_IN
- net N$13: now also U$2.XTAL_P; no longer U$1.XTAL_P
- net N$15: now also U$2.XTAL_N; no longer U$1.XTAL_N
- net U0RXD: now also J2.17, U$2.(GPIO3/CLK_OUT2/HS2_DATA0)U0RXD; no longer J2.20, U$1.(GPIO3/CLK_OUT2/HS2_DATA0)U0RXD
- net U0TXD: now also J2.18, U$2.(GPIO1/CLK_OUT3/HS2_DATA1)U0TXD; no longer J2.19, U$1.(GPIO1/CLK_OUT3/HS2_DATA1)U0TXD
Other:
- moved on the sheet: C1, C2, C5, R2

Commit message: Re-routing i/o traces to get better ground fill.
Parts:
- C27: value 3.3nF -> 3.0nF; device SparkFun-Capacitors:3.3NF-0603-100V-10% -> esp32-thing-temp:3.0NF-0603-50V-5%
- FD1, FD2: value FIDUCIAL1X2 -> FIDUCIALUFIDUCIAL; device SparkFun-Aesthetics:FIDUCIAL1X2 -> SparkFun-Aesthetics:FIDUCIALUFIDUCIAL
- LOGO3: value SFE_LOGO_NAME.1_INCH -> SFE_LOGO_NAME.2_INCH; device SparkFun-Aesthetics:SFE_LOGO_NAME.1_INCH -> SparkFun-Aesthetics:SFE_LOGO_NAME.2_INCH
- R2: value 14k -> 20k; device esp32-thing-temp:14KOHM-1/10W-1%(0603) -> SparkFun-Resistors:20KOHM-0603-1/10W-1%
Connections:
- net CAP_10N: now also U$2.CAP1; no longer U$2.CAP_10N
- net N$4: now also U$2.CAP2; no longer U$2.RES_14K
Other:
- note added: "v03"
- note removed: "v02"
- moved on the sheet: C1, C2, C27, R2
Changed lines of the file:
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@@
 <part name="C2" library="esp32-thing-temp" deviceset="270PF-50V-5%(0603)" device="" value="270pF"/>
 <part name="C5" library="SparkFun-Capacitors" deviceset="10NF" device="-0603-50V-10%" value="10nF"/>
-<part name="R2" library="esp32-thing-temp" deviceset="14KOHM-1/10W-1%(0603)" device="" value="14k"/>
+<part name="R2" library="SparkFun-Resistors" deviceset="20KOHM" device="-0603-1/10W-1%" value="20k"/>
 <part name="GND3" library="SparkFun-Aesthetics" deviceset="GND" device=""/>
 <part name="GND35" library="SparkFun-Aesthetics" deviceset="GND" device=""/>
@@
 <part name="GND37" library="SparkFun-Aesthetics" deviceset="GND" device=""/>
 <part name="LOGO2" library="SparkFun-Aesthetics" deviceset="OSHW-LOGO" device="MINI" value="OSHW-LOGOMINI"/>
-<part name="FD1" library="SparkFun-Aesthetics" deviceset="FIDUCIAL" device="1X2"/>
-<part name="FD2" library="SparkFun-Aesthetics" deviceset="FIDUCIAL" device="1X2"/>
+<part name="FD1" library="SparkFun-Aesthetics" deviceset="FIDUCIAL" device="UFIDUCIAL" value="FIDUCIALUFIDUCIAL"/>
+<part name="FD2" library="SparkFun-Aesthetics" deviceset="FIDUCIAL" device="UFIDUCIAL" value="FIDUCIALUFIDUCIAL"/>
 <part name="GND38" library="SparkFun-Aesthetics" deviceset="GND" device=""/>
 <part name="GND39" library="SparkFun-Aesthetics" deviceset="GND" device=""/>
@@
 <part name="SUPPLY6" library="SparkFun-Aesthetics" deviceset="V_BATT" device=""/>
 <part name="SUPPLY15" library="SparkFun-Aesthetics" deviceset="V_BATT" device=""/>
-<part name="LOGO3" library="SparkFun-Aesthetics" deviceset="SFE_LOGO_NAME" device=".1_INCH" value="SFE_LOGO_NAME.1_INCH"/>
+<part name="LOGO3" library="SparkFun-Aesthetics" deviceset="SFE_LOGO_NAME" device=".2_INCH" value="SFE_LOGO_NAME.2_INCH"/>
 <part name="R9" library="SparkFun-Resistors" deviceset="10KOHM-1/10W-1%(0603)" device="0603" value="10K"/>
 <part name="SUPPLY17" library="SparkFun-Aesthetics" deviceset="3.3V" device=""/>
 <part name="U$2" library="esp32-thing-temp" deviceset="ESP32-2" device=""/>
-<part name="C27" library="SparkFun-Capacitors" deviceset="3.3NF" device="-0603-100V-10%" value="3.3nF"/>
+<part name="C27" library="esp32-thing-temp" deviceset="3.0NF" device="-0603-50V-5%" value="3.0nF"/>
 <part name="GND40" library="SparkFun-Aesthetics" deviceset="GND" device=""/>
 </parts>
@@
 <text x="200.66" y="53.34" size="2.54" layer="94" align="top-left">GPIO5 LED</text>
 <text x="332.74" y="104.14" size="2.54" layer="94" align="top-left">Headers</text>
-<text x="421.64" y="10.16" size="2.54" layer="94" align="top-left">v02</text>
+<text x="421.64" y="10.16" size="2.54" layer="94" align="top-left">v03</text>
 <text x="354.838" y="11.43" size="2.54" layer="94" rot="MR180" align="top-left">Jim Lindblom</text>
 <text x="68.58" y="167.64" size="2.032" layer="97" font="vector" align="bottom-right">ESP32 VCC Range: 2.8-3.6V</text>
@@
 <attribute name="VALUE" x="50.8" y="124.206" size="1.778" layer="96" font="vector" rot="MR180"/>
 </instance>
-<instance part="C1" gate="G$1" x="40.64" y="99.06" smashed="yes" rot="R90">
-<attribute name="NAME" x="38.1" y="99.314" size="1.778" layer="95" rot="MR0"/>
-<attribute name="VALUE" x="40.64" y="99.314" size="1.778" layer="96"/>
-</instance>
-<instance part="C2" gate="G$1" x="40.64" y="91.44" smashed="yes" rot="MR270">
-<attribute name="NAME" x="38.1" y="91.186" size="1.778" layer="95" align="top-right"/>
-<attribute name="VALUE" x="40.64" y="91.186" size="1.778" layer="96" rot="MR180"/>
+<instance part="C1" gate="G$1" x="58.42" y="99.06" smashed="yes" rot="R90">
+<attribute name="NAME" x="55.88" y="99.314" size="1.778" layer="95" rot="MR0"/>
+<attribute name="VALUE" x="58.42" y="99.314" size="1.778" layer="96"/>
+</instance>
+<instance part="C2" gate="G$1" x="58.42" y="91.44" smashed="yes" rot="MR270">
+<attribute name="NAME" x="55.88" y="91.186" size="1.778" layer="95" align="top-right"/>
+<attribute name="VALUE" x="58.42" y="91.186" size="1.778" layer="96" rot="MR180"/>
 </instance>
 <instance part="C5" gate="G$1" x="48.26" y="78.74" rot="R180"/>
-<instance part="R2" gate="G$1" x="60.96" y="83.82" rot="R180"/>
+<instance part="R2" gate="G$1" x="60.96" y="81.28" rot="R180"/>
 <instance part="GND3" gate="1" x="48.26" y="63.5"/>
 <instance part="GND35" gate="1" x="236.22" y="129.54" rot="MR0"/>
@@
 <instance part="SUPPLY17" gate="G$1" x="299.72" y="91.44"/>
 <instance part="U$2" gate="G$1" x="124.46" y="116.84"/>
-<instance part="C27" gate="G$1" x="63.5" y="78.74" rot="MR270"/>
+<instance part="C27" gate="G$1" x="63.5" y="76.2" rot="MR270"/>
 <instance part="GND40" gate="1" x="71.12" y="63.5"/>
 </instances>
@@
 <pinref part="U$2" gate="G$1" pin="SENSOR_VN(GPI39/ADC1:3/RTC3)"/>
 <pinref part="C2" gate="G$1" pin="2"/>
-<wire x1="43.18" y1="91.44" x2="73.66" y2="91.44" width="0.1524" layer="91"/>
+<wire x1="60.96" y1="91.44" x2="73.66" y2="91.44" width="0.1524" layer="91"/>
 </segment>
 <segment>
@@
 <pinref part="U$2" gate="G$1" pin="SENSOR_CAPN(GPI38/ADC1:2/RTC2)"/>
 <pinref part="C2" gate="G$1" pin="1"/>
-<wire x1="33.02" y1="93.98" x2="33.02" y2="91.44" width="0.1524" layer="91"/>
-<wire x1="33.02" y1="91.44" x2="35.56" y2="91.44" width="0.1524" layer="91"/>
-<wire x1="73.66" y1="93.98" x2="33.02" y2="93.98" width="0.1524" layer="91"/>
+<wire x1="50.8" y1="93.98" x2="50.8" y2="91.44" width="0.1524" layer="91"/>
+<wire x1="50.8" y1="91.44" x2="53.34" y2="91.44" width="0.1524" layer="91"/>
+<wire x1="73.66" y1="93.98" x2="50.8" y2="93.98" width="0.1524" layer="91"/>
 </segment>
 <segment>
@@
 <segment>
 <pinref part="C1" gate="G$1" pin="2"/>
-<wire x1="43.18" y1="99.06" x2="73.66" y2="99.06" width="0.1524" layer="91"/>
+<wire x1="60.96" y1="99.06" x2="73.66" y2="99.06" width="0.1524" layer="91"/>
 <pinref part="U$2" gate="G$1" pin="SENSOR_VP(GPI36/ADC1:0/RTC0)"/>
 <label x="68.58" y="99.06" size="1.778" layer="95"/>
@@
 <segment>
 <pinref part="C1" gate="G$1" pin="1"/>
-<wire x1="35.56" y1="99.06" x2="33.02" y2="99.06" width="0.1524" layer="91"/>
-<wire x1="33.02" y1="99.06" x2="33.02" y2="96.52" width="0.1524" layer="91"/>
-<wire x1="33.02" y1="96.52" x2="73.66" y2="96.52" width="0.1524" layer="91"/>
+<wire x1="53.34" y1="99.06" x2="50.8" y2="99.06" width="0.1524" layer="91"/>
+<wire x1="50.8" y1="99.06" x2="50.8" y2="96.52" width="0.1524" layer="91"/>
+<wire x1="50.8" y1="96.52" x2="73.66" y2="96.52" width="0.1524" layer="91"/>
 <pinref part="U$2" gate="G$1" pin="SENSOR_CAPP(GPI37/ADC1:1/RTC1)"/>
 <label x="68.58" y="96.52" size="1.778" layer="95"/>
@@
 <wire x1="53.34" y1="86.36" x2="48.26" y2="86.36" width="0.1524" layer="91"/>
 <wire x1="48.26" y1="86.36" x2="48.26" y2="81.28" width="0.1524" layer="91"/>
-<pinref part="U$2" gate="G$1" pin="CAP_10N"/>
+<pinref part="U$2" gate="G$1" pin="CAP1"/>
 <pinref part="C27" gate="G$1" pin="1"/>
-<wire x1="58.42" y1="78.74" x2="53.34" y2="78.74" width="0.1524" layer="91"/>
-<wire x1="53.34" y1="78.74" x2="53.34" y2="83.82" width="0.1524" layer="91"/>
+<wire x1="58.42" y1="76.2" x2="53.34" y2="76.2" width="0.1524" layer="91"/>
+<wire x1="53.34" y1="76.2" x2="53.34" y2="81.28" width="0.1524" layer="91"/>
 <junction x="53.34" y="86.36"/>
 <pinref part="R2" gate="G$1" pin="2"/>
-<wire x1="53.34" y1="83.82" x2="53.34" y2="86.36" width="0.1524" layer="91"/>
-<wire x1="55.88" y1="83.82" x2="53.34" y2="83.82" width="0.1524" layer="91"/>
-<junction x="53.34" y="83.82"/>
+<wire x1="53.34" y1="81.28" x2="53.34" y2="86.36" width="0.1524" layer="91"/>
+<wire x1="55.88" y1="81.28" x2="53.34" y2="81.28" width="0.1524" layer="91"/>
+<junction x="53.34" y="81.28"/>
 </segment>
 </net>
@@
 <segment>
 <pinref part="C27" gate="G$1" pin="2"/>
-<wire x1="66.04" y1="78.74" x2="68.58" y2="78.74" width="0.1524" layer="91"/>
-<wire x1="68.58" y1="78.74" x2="68.58" y2="83.82" width="0.1524" layer="91"/>
-<pinref part="U$2" gate="G$1" pin="RES_14K"/>
+<wire x1="66.04" y1="76.2" x2="68.58" y2="76.2" width="0.1524" layer="91"/>
+<wire x1="68.58" y1="76.2" x2="68.58" y2="81.28" width="0.1524" layer="91"/>
+<pinref part="U$2" gate="G$1" pin="CAP2"/>
+<wire x1="68.58" y1="81.28" x2="68.58" y2="83.82" width="0.1524" layer="91"/>
 <wire x1="68.58" y1="83.82" x2="73.66" y2="83.82" width="0.1524" layer="91"/>
 <pinref part="R2" gate="G$1" pin="1"/>
-<wire x1="66.04" y1="83.82" x2="68.58" y2="83.82" width="0.1524" layer="91"/>
-<junction x="68.58" y="83.82"/>
-</segment>
-</net>
+<wire x1="66.04" y1="81.28" x2="68.58" y2="81.28" width="0.1524" layer="91"/>
+<junction x="68.58" y="81.28"/>
+</segment>
+</net>

Commit message: Post-review fixes - changed C18 to 100pF
Parts:
- C18: value 0.1uF -> 100pF; device SparkFun-Capacitors:0.1UF-0603-25V-(+80/-20%) -> SparkFun-Capacitors:100PF-0603-50V-5%
- R1, R9: value 10K -> 10k
Other:
- note added: "CHIP_PU is the ESP32's enable/reset pin. It must be pulled high to turn the ESP32 on."
- note added: "Near VDDA 46, 43"
- note added: "Near VDDA3P3 3, 4"
- note added: "Near VDDPST_SDIO 26"
- note removed: "Near VDDA 46"
- note removed: "Near VDDA3P3 3/4"
- note removed: "Near VDDPST_SDIO 25"
Changed lines of the file:
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@@
 <part name="S1" library="SparkFun-Electromechanical" deviceset="SWITCH-MOMENTARY-2" device="SMD-4.6X2.8MM" value="RESET"/>
 <part name="GND1" library="SparkFun-Aesthetics" deviceset="GND" device=""/>
-<part name="R1" library="SparkFun-Resistors" deviceset="10KOHM-1/10W-1%(0603)" device="0603" value="10K"/>
+<part name="R1" library="SparkFun-Resistors" deviceset="10KOHM-1/10W-1%(0603)" device="0603" value="10k"/>
 <part name="SUPPLY2" library="SparkFun-Aesthetics" deviceset="3.3V" device=""/>
 <part name="GND2" library="SparkFun-Aesthetics" deviceset="GND" device=""/>
@@
 <part name="R18" library="SparkFun-Resistors" deviceset="10KOHM" device="-0603-1/10W-1%" value="10k"/>
 <part name="SUPPLY8" library="SparkFun-Aesthetics" deviceset="3.3V" device=""/>
-<part name="C18" library="SparkFun-Capacitors" deviceset="0.1UF" device="-0603-25V-(+80/-20%)" value="0.1uF"/>
+<part name="C18" library="SparkFun-Capacitors" deviceset="100PF" device="-0603-50V-5%" value="100pF"/>
 <part name="SUPPLY9" library="SparkFun-Aesthetics" deviceset="3.3V" device=""/>
 <part name="GND5" library="SparkFun-Aesthetics" deviceset="GND" device=""/>
@@
 <part name="SUPPLY15" library="SparkFun-Aesthetics" deviceset="V_BATT" device=""/>
 <part name="LOGO3" library="SparkFun-Aesthetics" deviceset="SFE_LOGO_NAME" device=".2_INCH" value="SFE_LOGO_NAME.2_INCH"/>
-<part name="R9" library="SparkFun-Resistors" deviceset="10KOHM-1/10W-1%(0603)" device="0603" value="10K"/>
+<part name="R9" library="SparkFun-Resistors" deviceset="10KOHM-1/10W-1%(0603)" device="0603" value="10k"/>
 <part name="SUPPLY17" library="SparkFun-Aesthetics" deviceset="3.3V" device=""/>
 <part name="U$2" library="esp32-thing-temp" deviceset="ESP32-2" device=""/>
@@
 <sheet>
 <plain>
-<text x="355.6" y="160.02" size="1.905" layer="91" font="vector">Boot Mode Configuration
+<text x="355.6" y="160.02" size="1.905" layer="97" font="vector">Boot Mode Configuration
 Pin        Default     Boot   Download
 GPIO0        1         1       0
@@
 <text x="332.74" y="190.5" size="2.54" layer="94" align="top-left">Auto-Reset</text>
 <text x="40.64" y="38.1" size="1.27" layer="97" align="bottom-center">Near VDDA
-46</text>
+46, 43</text>
 <text x="60.96" y="38.1" size="1.27" layer="97" align="bottom-center">Near VDDA_LNA
 1</text>
-<text x="81.28" y="38.1" size="1.27" layer="97" align="bottom-center">Near VDDA3P3
-3/4</text>
+<text x="91.44" y="38.1" size="1.27" layer="97" align="bottom-center">Near VDDA3P3
+3, 4</text>
 <wire x1="50.8" y1="40.64" x2="50.8" y2="12.7" width="0.2032" layer="97" style="shortdash"/>
 <wire x1="71.12" y1="40.64" x2="71.12" y2="12.7" width="0.2032" layer="97" style="shortdash"/>
@@
 <wire x1="127" y1="40.64" x2="127" y2="12.7" width="0.2032" layer="97" style="shortdash"/>
 <text x="137.16" y="38.1" size="1.27" layer="97" align="bottom-center">Near VDDPST_SDIO
-25</text>
+26</text>
 <wire x1="147.32" y1="40.64" x2="147.32" y2="12.7" width="0.2032" layer="97" style="shortdash"/>
 <text x="157.48" y="38.1" size="1.27" layer="97" align="bottom-center">Near VDDPST_RTC
@@
 <text x="421.64" y="10.16" size="2.54" layer="94" align="top-left">v03</text>
 <text x="354.838" y="11.43" size="2.54" layer="94" rot="MR180" align="top-left">Jim Lindblom</text>
-<text x="68.58" y="167.64" size="2.032" layer="97" font="vector" align="bottom-right">ESP32 VCC Range: 2.8-3.6V</text>
+<text x="124.46" y="165.1" size="2.032" layer="97" font="vector" align="bottom-center">ESP32 VCC Range: 2.8-3.6V</text>
 <text x="274.32" y="162.56" size="2.032" layer="97" font="vector">SJ3 allows selection between
 FLASH_VDD and 3.3V as the
@@
 <text x="381" y="114.3" size="1.778" layer="97" font="vector" align="top-center">If DTR is LOW, toggling RTS from HIGH to LOW resets to run mode.
 If RTS is HIGH, toggling DTR from LOW to HIGH resets to bootloader.</text>
+<text x="58.42" y="152.4" size="1.27" layer="97" rot="MR0">CHIP_PU is the ESP32's enable/reset pin.
+It must be pulled high to turn the ESP32 on.</text>
+<wire x1="58.42" y1="152.4" x2="61.468" y2="143.51" width="0.2032" layer="97"/>
 </plain>
 <instances>

Commit message: Post-checklist fixes.
Changed lines of the file:
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@@
 <part name="C27" library="esp32-thing-temp" deviceset="3.0NF" device="-0603-50V-5%" value="3.0nF"/>
 <part name="GND40" library="SparkFun-Aesthetics" deviceset="GND" device=""/>
+<part name="GND42" library="SparkFun-PowerSymbols" deviceset="GND" device=""/>
 </parts>
 <sheets>
@@
 <instance part="C27" gate="G$1" x="63.5" y="76.2" rot="MR270"/>
 <instance part="GND40" gate="1" x="71.12" y="63.5"/>
+<instance part="GND42" gate="1" x="421.64" y="88.9"/>
 </instances>
 <busses>
@@
 </segment>
 <segment>
-<wire x1="406.4" y1="93.98" x2="408.94" y2="93.98" width="0.1524" layer="91"/>
-<label x="408.94" y="93.98" size="1.27" layer="95" xref="yes"/>
 <pinref part="J2" gate="G$1" pin="20"/>
+<pinref part="GND42" gate="1" pin="GND"/>
+<wire x1="406.4" y1="93.98" x2="421.64" y2="93.98" width="0.1524" layer="91"/>
+<wire x1="421.64" y1="93.98" x2="421.64" y2="91.44" width="0.1524" layer="91"/>
 </segment>
 </net>
